Commit message: fix: Update the stop and go logic for traffic light
Deep copy base_waypoint to keep the main one untouched

File: ros/src/dbw_mkz_description/urdf/mkz_13_structure.urdf.xacro (robot description, xacro)
@@ -5,5 +5,5 @@
     <link name="base_link">
     </link>
-    <link name="base_fix_link">
+    <link name="base_fixed_link">
       <inertial>
         <origin xyz="1.4225 0 0.25" rpy="0 0 0"/>
@@ -119,24 +119,24 @@
       </collision>
     </link>
-    <joint name="base_fix_link_joint" type="fixed">
+    <joint name="base_link" type="fixed">
       <origin xyz="0 0 0.33" rpy="0 0 0"/>
       <parent link="base_link"/>
-      <child link="base_fix_link"/>
+      <child link="base_fixed_link"/>
     </joint>
-    <joint name="steer_fl_joint" type="revolute">
+    <joint name="steer_fl" type="revolute">
       <origin xyz="2.85 0.79121 0.0" rpy="0 0 0"/>
-      <parent link="base_fix_link"/>
+      <parent link="base_fixed_link"/>
       <child link="steer_fl"/>
       <axis xyz="0 0 1.0"/>
       <limit lower="-0.6" upper="0.6" effort="0" velocity="0"/>
     </joint>
-    <joint name="steer_fr_joint" type="revolute">
+    <joint name="steer_fr" type="revolute">
       <origin xyz="2.85 -0.79121 0.0" rpy="0 0 0"/>
-      <parent link="base_fix_link"/>
+      <parent link="base_fixed_link"/>
       <child link="steer_fr"/>
       <axis xyz="0 0 1.0"/>
       <limit lower="-0.6" upper="0.6" effort="0" velocity="0"/>
     </joint>
-    <joint name="wheel_fl_joint" type="continuous">
+    <joint name="wheel_fl" type="continuous">
       <origin xyz="0 0 0" rpy="1.570796 0 -3.141593"/>
       <parent link="steer_fl"/>
@@ -145,5 +145,5 @@
       <limit effort="0" velocity="22.0"/>
     </joint>
-    <joint name="wheel_fr_joint" type="continuous">
+    <joint name="wheel_fr" type="continuous">
       <origin xyz="0 0 0" rpy="1.570796 0 -3.141593"/>
       <parent link="steer_fr"/>
@@ -152,14 +152,14 @@
       <limit effort="0" velocity="22.0"/>
     </joint>
-    <joint name="wheel_rl_joint" type="continuous">
+    <joint name="wheel_rl" type="continuous">
       <origin xyz="0 0.7874 0" rpy="1.570796 0 -3.141593"/>
-      <parent link="base_fix_link"/>
+      <parent link="base_fixed_link"/>
       <child link="wheel_rl"/>
       <axis xyz="0 0 1.0"/>
       <limit effort="5000.0" velocity="22.0"/>
     </joint>
-    <joint name="wheel_rr_joint" type="continuous">
+    <joint name="wheel_rr" type="continuous">
       <origin xyz="0 -0.7874 0" rpy="1.570796 0 -3.141593"/>
-      <parent link="base_fix_link"/>
+      <parent link="base_fixed_link"/>
       <child link="wheel_rr"/>
       <axis xyz="0 0 1.0"/>
